File: hw/wifi_car/untitled.sch (EAGLE design)
At the start: 54 parts, among them IC1 LPC1114FBD48, U1 MCP16301T-I/CHY

Commit message: Added ADC for battery measurements
Parts:
- removed SW_RESET: (no value), wirepad:SMD2
- added SW_RES, TP1: TPB1,27, testpad:TPB1,27
- SWCLK, SWDIO, VDD: value (none) -> TPB1,27; device wirepad:SMD2 -> testpad:TPB1,27
Connections:
- removed net LED10: IC1.PIO0_6/USB_CONNECT/SCK, LED7.C
- removed net LED12: IC1.PIO2_9, LED8.C
- new net N$18: IC1.PIO0_1/CLKOUT/CT32B0_MAT2/USB_FTOGGLE, TP1.TP
- net LED2: now also IC1.PIO0_4/SCL, LED2.C; no longer IC1.PIO0_3/USB_VBUS
- net LED3: now also IC1.PIO1_9/CT16B1_MAT0, LED3.C; no longer IC1.PIO0_4/SCL, LED2.C
- net LED4: now also IC1.PIO3_4, LED4.C; no longer IC1.PIO0_5/SDA
- net LED5: now also IC1.PIO2_4, LED5.C; no longer IC1.PIO1_9/CT16B1_MAT0, LED3.C
- net LED6: now also IC1.PIO2_5, LED6.C; no longer IC1.PIO3_4, LED4.C
- net LED7: now also IC1.PIO0_6/USB_CONNECT/SCK, LED7.C; no longer IC1.PIO2_4, LED5.C
- net LED8: now also IC1.PIO2_9, LED8.C; no longer IC1.PIO2_5, LED6.C
- net PWM12: now also SWCLK.TP; no longer SWCLK.P
- net PWM2: now also SWDIO.TP; no longer SWDIO.P
- net SW_RESET: now also SW_RES.TP; no longer SW_RESET.P
- net VDD: now also VDD.TP; no longer VDD.P

Commit message: Board and schematic update
Parts:
- removed PAD1, PAD2: (no value), wirepad:SMD2
- added C7, C8, C9: 10u, rcl:C-EUC0805
- added R18: 11k, rcl:R-EU_R0805
- R9: value (none) -> 34k; device rcl:R-EU_R0603 -> rcl:R-EU_R0805
Connections:
- removed net LED11: IC1.PIO0_7/CTS
- removed net LED9: IC1.PIO3_5
- removed net N$7: JP2.8, PAD1.P
- removed net N$9: BAT+.P, R9.2, U1.EN, U1.VIN
- new net ADC: IC1.PIO1_10/AD6/CT16B1_MAT1, R18.2, R9.1
- net BAT+: now also BAT+.P, C7.2, R9.2, U1.EN, U1.VIN
- net GND: now also C7.1, C8.1, C9.1, R18.1; no longer R9.1
- net VDD: now also C8.2, C9.2, JP2.8; no longer PAD2.P
Other:
- moved on the sheet: R9
Changed lines of the file:
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@@
 <part name="C6" library="rcl" deviceset="C-EU" device="C0805" value="100n"/>
 <part name="D1" library="diode" deviceset="SCHOTTKY-DIODE" device="SMD"/>
-<part name="R9" library="rcl" deviceset="R-EU_" device="R0603"/>
 <part name="GND12" library="supply1" deviceset="GND" device=""/>
 <part name="GND13" library="supply1" deviceset="GND" device=""/>
@@
 <part name="BAT+" library="wirepad" deviceset="SMD5" device=""/>
 <part name="BAT-" library="wirepad" deviceset="SMD5" device=""/>
-<part name="PAD1" library="wirepad" deviceset="SMD2" device=""/>
-<part name="PAD2" library="wirepad" deviceset="SMD2" device=""/>
 <part name="LED1" library="led" deviceset="LED" device="CHIP-LED0805"/>
 <part name="R11" library="rcl" deviceset="R-EU_" device="R0805"/>
@@
 <part name="SWDIO" library="testpad" deviceset="TP" device="B1,27"/>
 <part name="SW_RES" library="testpad" deviceset="TP" device="B1,27"/>
+<part name="C7" library="rcl" deviceset="C-EU" device="C0805" value="10u"/>
+<part name="C8" library="rcl" deviceset="C-EU" device="C0805" value="10u"/>
+<part name="C9" library="rcl" deviceset="C-EU" device="C0805" value="10u"/>
+<part name="GND11" library="supply1" deviceset="GND" device=""/>
+<part name="R9" library="rcl" deviceset="R-EU_" device="R0805" value="34k"/>
+<part name="R18" library="rcl" deviceset="R-EU_" device="R0805" value="11k"/>
+<part name="GND16" library="supply1" deviceset="GND" device=""/>
 </parts>
 <sheets>
@@
 <instance part="GND9" gate="1" x="198.12" y="7.62"/>
 <instance part="GND10" gate="1" x="218.44" y="7.62"/>
-<instance part="PAD1" gate="1" x="220.98" y="91.44" rot="R270"/>
-<instance part="PAD2" gate="1" x="231.14" y="93.98" rot="R90"/>
 <instance part="LED1" gate="G$1" x="30.48" y="-53.34"/>
 <instance part="R11" gate="G$1" x="30.48" y="-43.18" rot="R90"/>
@@
 </segment>
 <segment>
-<pinref part="VDD3" gate="G$1" pin="VDD"/>
-<pinref part="PAD2" gate="1" pin="P"/>
-</segment>
-<segment>
 <pinref part="VDD10" gate="G$1" pin="VDD"/>
 <pinref part="R11" gate="G$1" pin="2"/>
@@
 <pinref part="R17" gate="G$1" pin="2"/>
 <wire x1="101.6" y1="-38.1" x2="101.6" y2="-35.56" width="0.1524" layer="91"/>
+</segment>
+<segment>
+<pinref part="JP2" gate="A" pin="8"/>
+<wire x1="213.36" y1="88.9" x2="231.14" y2="88.9" width="0.1524" layer="91"/>
+<pinref part="VDD3" gate="G$1" pin="VDD"/>
+<wire x1="231.14" y1="88.9" x2="231.14" y2="96.52" width="0.1524" layer="91"/>
 </segment>
 </net>
@@
 <pinref part="IC1" gate="G$1" pin="SWCLK/PIO0_10/SCK/CT16B0_MAT2"/>
 <wire x1="38.1" y1="58.42" x2="22.86" y2="58.42" width="0.1524" layer="91"/>
-<label x="2.54" y="58.42" size="1.778" layer="95" rot="R180" xref="yes"/>
 <pinref part="SWCLK" gate="G$1" pin="TP"/>
-<wire x1="22.86" y1="58.42" x2="2.54" y2="58.42" width="0.1524" layer="91"/>
-<junction x="22.86" y="58.42"/>
 </segment>
 </net>
@@
 </segment>
 </net>
-<net name="N$7" class="0">
-<segment>
-<pinref part="JP2" gate="A" pin="8"/>
-<wire x1="213.36" y1="88.9" x2="220.98" y2="88.9" width="0.1524" layer="91"/>
-<wire x1="220.98" y1="88.9" x2="223.52" y2="88.9" width="0.1524" layer="91"/>
-<pinref part="PAD1" gate="1" pin="P"/>
-<junction x="220.98" y="88.9"/>
-</segment>
-</net>
 <net name="LED1" class="0">
 <segment>
@@
 </segment>
 </net>
-<net name="LED9" class="0">
-<segment>
-<pinref part="IC1" gate="G$1" pin="PIO3_5"/>
-<wire x1="132.08" y1="5.08" x2="132.08" y2="0" width="0.1524" layer="91"/>
-<wire x1="132.08" y1="0" x2="144.78" y2="0" width="0.1524" layer="91"/>
-<label x="144.78" y="0" size="1.778" layer="95" xref="yes"/>
-</segment>
-</net>
 <net name="LED2" class="0">
 <segment>
@@
 <wire x1="91.44" y1="-58.42" x2="91.44" y2="-60.96" width="0.1524" layer="91"/>
 <label x="91.44" y="-60.96" size="1.778" layer="95" rot="R270" xref="yes"/>
-</segment>
-</net>
-<net name="LED11" class="0">
-<segment>
-<pinref part="IC1" gate="G$1" pin="PIO0_7/CTS"/>
-<label x="10.16" y="66.04" size="1.778" layer="95" rot="R180" xref="yes"/>
-<wire x1="38.1" y1="66.04" x2="10.16" y2="66.04" width="0.1524" layer="91"/>
 </segment>
 </net>
@@
 <wire x1="33.02" y1="78.74" x2="7.62" y2="78.74" width="0.1524" layer="91"/>
 <pinref part="TP1" gate="G$1" pin="TP"/>
+</segment>
+</net>
+<net name="ADC" class="0">
+<segment>
+<pinref part="IC1" gate="G$1" pin="PIO1_10/AD6/CT16B1_MAT1"/>
+<wire x1="132.08" y1="58.42" x2="142.24" y2="58.42" width="0.1524" layer="91"/>
+<wire x1="142.24" y1="58.42" x2="142.24" y2="55.88" width="0.1524" layer="91"/>
+<wire x1="142.24" y1="55.88" x2="144.78" y2="55.88" width="0.1524" layer="91"/>
+<label x="144.78" y="55.88" size="1.778" layer="95" xref="yes"/>
 </segment>
 </net>
@@
 <instance part="C6" gate="G$1" x="81.28" y="58.42" rot="R180"/>
 <instance part="D1" gate="G$1" x="86.36" y="50.8" rot="R90"/>
-<instance part="R9" gate="G$1" x="35.56" y="48.26" rot="R90"/>
 <instance part="GND12" gate="1" x="86.36" y="45.72"/>
 <instance part="GND13" gate="1" x="111.76" y="22.86"/>
@@
 <instance part="BAT+" gate="1" x="25.4" y="53.34"/>
 <instance part="BAT-" gate="1" x="40.64" y="33.02"/>
+<instance part="C7" gate="G$1" x="35.56" y="48.26" rot="R180"/>
+<instance part="C8" gate="G$1" x="121.92" y="45.72" rot="R180"/>
+<instance part="C9" gate="G$1" x="129.54" y="45.72" rot="R180"/>
+<instance part="GND11" gate="1" x="124.46" y="38.1"/>
+<instance part="R9" gate="G$1" x="58.42" y="12.7" rot="R90"/>
+<instance part="R18" gate="G$1" x="58.42" y="0" rot="R90"/>
+<instance part="GND16" gate="1" x="58.42" y="-10.16"/>
 </instances>
 <busses>
@@
 </segment>
 <segment>
-<pinref part="R9" gate="G$1" pin="1"/>
-<pinref part="GND15" gate="1" pin="GND"/>
-</segment>
-<segment>
 <pinref part="GND14" gate="1" pin="GND"/>
 <wire x1="43.18" y1="30.48" x2="43.18" y2="33.02" width="0.1524" layer="91"/>
@@
 <junction x="43.18" y="33.02"/>
 </segment>
-</net>
-<net name="N$9" class="0">
+<segment>
+<pinref part="GND15" gate="1" pin="GND"/>
+<pinref part="C7" gate="G$1" pin="1"/>
+<wire x1="35.56" y1="43.18" x2="35.56" y2="45.72" width="0.1524" layer="91"/>
+</segment>
+<segment>
+<pinref part="C8" gate="G$1" pin="1"/>
+<pinref part="C9" gate="G$1" pin="1"/>
+<wire x1="121.92" y1="43.18" x2="124.46" y2="43.18" width="0.1524" layer="91"/>
+<wire x1="124.46" y1="43.18" x2="129.54" y2="43.18" width="0.1524" layer="91"/>
+<wire x1="124.46" y1="43.18" x2="124.46" y2="40.64" width="0.1524" layer="91"/>
+<junction x="124.46" y="43.18"/>
+<pinref part="GND11" gate="1" pin="GND"/>
+</segment>
+<segment>
+<pinref part="R18" gate="G$1" pin="1"/>
+<wire x1="58.42" y1="-5.08" x2="58.42" y2="-7.62" width="0.1524" layer="91"/>
+<pinref part="GND16" gate="1" pin="GND"/>
+</segment>
+</net>
+<net name="BAT+" class="0">
 <segment>
 <pinref part="U1" gate="A" pin="VIN"/>
 <wire x1="45.72" y1="53.34" x2="40.64" y2="53.34" width="0.1524" layer="91"/>
-<pinref part="R9" gate="G$1" pin="2"/>
-<junction x="35.56" y="53.34"/>
 <wire x1="40.64" y1="53.34" x2="35.56" y2="53.34" width="0.1524" layer="91"/>
-<wire x1="35.56" y1="53.34" x2="27.94" y2="53.34" width="0.1524" layer="91"/>
 <pinref part="U1" gate="A" pin="EN"/>
+<wire x1="35.56" y1="53.34" x2="30.48" y2="53.34" width="0.1524" layer="91"/>
+<wire x1="30.48" y1="53.34" x2="27.94" y2="53.34" width="0.1524" layer="91"/>
 <wire x1="45.72" y1="48.26" x2="40.64" y2="48.26" width="0.1524" layer="91"/>
 <wire x1="40.64" y1="48.26" x2="40.64" y2="53.34" width="0.1524" layer="91"/>
 <junction x="40.64" y="53.34"/>
 <pinref part="BAT+" gate="1" pin="P"/>
+<pinref part="C7" gate="G$1" pin="2"/>
+<junction x="35.56" y="53.34"/>
+<pinref part="R9" gate="G$1" pin="2"/>
+<wire x1="58.42" y1="17.78" x2="30.48" y2="17.78" width="0.1524" layer="91"/>
+<wire x1="30.48" y1="17.78" x2="30.48" y2="53.34" width="0.1524" layer="91"/>
+<junction x="30.48" y="53.34"/>
+<label x="30.48" y="43.18" size="1.778" layer="95" rot="R180" xref="yes"/>
 </segment>
 </net>
@@
 <wire x1="111.76" y1="63.5" x2="99.06" y2="63.5" width="0.1524" layer="91"/>
 <pinref part="VDD9" gate="G$1" pin="VDD"/>
-</segment>
-</net>
+<pinref part="C8" gate="G$1" pin="2"/>
+<pinref part="C9" gate="G$1" pin="2"/>
+<wire x1="121.92" y1="50.8" x2="124.46" y2="50.8" width="0.1524" layer="91"/>
+<wire x1="124.46" y1="50.8" x2="129.54" y2="50.8" width="0.1524" layer="91"/>
+<wire x1="121.92" y1="50.8" x2="111.76" y2="50.8" width="0.1524" layer="91"/>
+<junction x="111.76" y="50.8"/>
+<junction x="121.92" y="50.8"/>
+<junction x="129.54" y="50.8"/>
+</segment>
+</net>
+<net name="ADC" class="0">
+<segment>
+<pinref part="R9" gate="G$1" pin="1"/>
+<pinref part="R18" gate="G$1" pin="2"/>
+<wire x1="58.42" y1="7.62" x2="58.42" y2="5.08" width="0.1524" layer="91"/>
+<wire x1="58.42" y1="5.08" x2="53.34" y2="5.08" width="0.1524" layer="91"/>
+<junction x="58.42" y="5.08"/>
+<label x="53.34" y="5.08" size="1.778" layer="95" rot="R180" xref="yes"/>
+</segment>
+</net>
